File: fsd-amp.kicad_pcb (KiCad board)
At the start: 2 copper layers, 13 parts, among them J1001 Screw_Terminal_01x06, J1004 AudioJack2_Ground_Switch, Q1001 FZT 653 ZET, Q1002 FZT 653 ZET, Q1003 FZT 753 ZET

Commit message: export footprints and symbols to project libraries
Parts:
- C1001, C1003: footprint Capacitor_THT:CP_Radial_D10.0mm_P5.00mm -> fp:CP_Radial_D10.0mm_P5.00mm
- C1002: footprint Capacitor_THT:C_Rect_L7.2mm_W11.0mm_P5.00mm_FKS2_FKP2_MKS2_MKP2 -> fp:C_Rect_L7.2mm_W11.0mm_P5.00mm_FKS2_FKP2_MKS2_MKP2
- D1001, D1002: footprint Diode_THT:D_DO-41_SOD81_P10.16mm_Horizontal -> fp:D_DO-41_SOD81_P10.16mm_Horizontal
- J1001: footprint TerminalBlock_MetzConnect:TerminalBlock_MetzConnect_Type101_RT01606HBWC_1x06_P5.08mm_Horizontal -> fp:TerminalBlock_MetzConnect_Type101_RT01606HBWC_1x06_P5.08mm_Horizontal
- J1004: footprint Connector_Audio:Jack_3.5mm_Ledino_KB3SPRS_Horizontal -> fp:Jack_3.5mm_Ledino_KB3SPRS_Horizontal
- Q1001, Q1002, Q1003: footprint Package_TO_SOT_SMD:SOT-223-3_TabPin2 -> fp:SOT-223-3_TabPin2
- R1001, R1002: footprint Resistor_THT:R_Axial_DIN0207_L6.3mm_D2.5mm_P10.16mm_Horizontal -> fp:R_Axial_DIN0207_L6.3mm_D2.5mm_P10.16mm_Horizontal
- RV1001: footprint Potentiometer_THT:Potentiometer_Bourns_3296W_Vertical -> fp:Potentiometer_Bourns_3296W_Vertical
Changed lines of the file:
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@@
 	(net 9 "Net-(D1002-K)")
 	(net 10 "/amp_in")
-	(footprint "Capacitor_THT:CP_Radial_D10.0mm_P5.00mm"
+	(footprint "fp:CP_Radial_D10.0mm_P5.00mm"
 		(layer "F.Cu")
 		(at 142.044646 102.02)
@@
 			)
 		)
-		(property "Footprint" "Capacitor_THT:CP_Radial_D10.0mm_P5.00mm"
+		(property "Footprint" "fp:CP_Radial_D10.0mm_P5.00mm"
 			(at 0 0 0)
 			(unlocked yes)
@@
 		)
 	)
-	(footprint "Potentiometer_THT:Potentiometer_Bourns_3296W_Vertical"
+	(footprint "fp:Potentiometer_Bourns_3296W_Vertical"
 		(layer "F.Cu")
 		(at 146.63 111.02)
@@
 			)
 		)
-		(property "Footprint" "Potentiometer_THT:Potentiometer_Bourns_3296W_Vertical"
+		(property "Footprint" "fp:Potentiometer_Bourns_3296W_Vertical"
 			(at 0 0 0)
 			(unlocked yes)
@@
 		)
 	)
-	(footprint "Capacitor_THT:C_Rect_L7.2mm_W11.0mm_P5.00mm_FKS2_FKP2_MKS2_MKP2"
+	(footprint "fp:C_Rect_L7.2mm_W11.0mm_P5.00mm_FKS2_FKP2_MKS2_MKP2"
 		(layer "F.Cu")
 		(at 165.5 114)
@@
 			)
 		)
-		(property "Footprint" "Capacitor_THT:C_Rect_L7.2mm_W11.0mm_P5.00mm_FKS2_FKP2_MKS2_MKP2"
+		(property "Footprint" "fp:C_Rect_L7.2mm_W11.0mm_P5.00mm_FKS2_FKP2_MKS2_MKP2"
 			(at 0 0 0)
 			(unlocked yes)
@@
 		)
 	)
-	(footprint "Capacitor_THT:CP_Radial_D10.0mm_P5.00mm"
+	(footprint "fp:CP_Radial_D10.0mm_P5.00mm"
 		(layer "F.Cu")
 		(at 142.044646 90.47)
@@
 			)
 		)
-		(property "Footprint" "Capacitor_THT:CP_Radial_D10.0mm_P5.00mm"
+		(property "Footprint" "fp:CP_Radial_D10.0mm_P5.00mm"
 			(at 0 0 0)
 			(unlocked yes)
@@
 		)
 	)
-	(footprint "Resistor_THT:R_Axial_DIN0207_L6.3mm_D2.5mm_P10.16mm_Horizontal"
+	(footprint "fp:R_Axial_DIN0207_L6.3mm_D2.5mm_P10.16mm_Horizontal"
 		(layer "F.Cu")
 		(at 151.89 113.8)
@@
 			)
 		)
-		(property "Footprint" "Resistor_THT:R_Axial_DIN0207_L6.3mm_D2.5mm_P10.16mm_Horizontal"
+		(property "Footprint" "fp:R_Axial_DIN0207_L6.3mm_D2.5mm_P10.16mm_Horizontal"
 			(at 0 0 0)
 			(unlocked yes)
@@
 		)
 	)
-	(footprint "Resistor_THT:R_Axial_DIN0207_L6.3mm_D2.5mm_P10.16mm_Horizontal"
+	(footprint "fp:R_Axial_DIN0207_L6.3mm_D2.5mm_P10.16mm_Horizontal"
 		(layer "F.Cu")
 		(at 151.89 109.75)
@@
 			)
 		)
-		(property "Footprint" "Resistor_THT:R_Axial_DIN0207_L6.3mm_D2.5mm_P10.16mm_Horizontal"
+		(property "Footprint" "fp:R_Axial_DIN0207_L6.3mm_D2.5mm_P10.16mm_Horizontal"
 			(at 0 0 0)
 			(unlocked yes)
@@
 		)
 	)
-	(footprint "Connector_Audio:Jack_3.5mm_Ledino_KB3SPRS_Horizontal"
+	(footprint "fp:Jack_3.5mm_Ledino_KB3SPRS_Horizontal"
 		(layer "F.Cu")
 		(at 160.64 96.62)
@@
 			)
 		)
-		(property "Footprint" "Connector_Audio:Jack_3.5mm_Ledino_KB3SPRS_Horizontal"
+		(property "Footprint" "fp:Jack_3.5mm_Ledino_KB3SPRS_Horizontal"
 			(at 0 0 0)
 			(unlocked yes)
@@
 		)
 	)
-	(footprint "Package_TO_SOT_SMD:SOT-223-3_TabPin2"
+	(footprint "fp:SOT-223-3_TabPin2"
 		(layer "F.Cu")
 		(at 133.58 88.895)
@@
 			)
 		)
-		(property "Footprint" "Package_TO_SOT_SMD:SOT-223-3_TabPin2"
+		(property "Footprint" "fp:SOT-223-3_TabPin2"
 			(at 0 0 0)
 			(unlocked yes)
@@
 		)
 	)
-	(footprint "Package_TO_SOT_SMD:SOT-223-3_TabPin2"
+	(footprint "fp:SOT-223-3_TabPin2"
 		(layer "F.Cu")
 		(at 133.58 97.22)
@@
 			)
 		)
-		(property "Footprint" "Package_TO_SOT_SMD:SOT-223-3_TabPin2"
+		(property "Footprint" "fp:SOT-223-3_TabPin2"
 			(at 0 0 0)
 			(unlocked yes)
@@
 		)
 	)
-	(footprint "Package_TO_SOT_SMD:SOT-223-3_TabPin2"
+	(footprint "fp:SOT-223-3_TabPin2"
 		(layer "F.Cu")
 		(at 133.58 105.545)
@@
 			)
 		)
-		(property "Footprint" "Package_TO_SOT_SMD:SOT-223-3_TabPin2"
+		(property "Footprint" "fp:SOT-223-3_TabPin2"
 			(at 0 0 0)
 			(unlocked yes)
@@
 		)
 	)
-	(footprint "Diode_THT:D_DO-41_SOD81_P10.16mm_Horizontal"
+	(footprint "fp:D_DO-41_SOD81_P10.16mm_Horizontal"
 		(layer "F.Cu")
 		(at 152.19 105.6)
@@
 			)
 		)
-		(property "Footprint" "Diode_THT:D_DO-41_SOD81_P10.16mm_Horizontal"
+		(property "Footprint" "fp:D_DO-41_SOD81_P10.16mm_Horizontal"
 			(at 0 0 0)
 			(unlocked yes)
@@
 		)
 	)
-	(footprint "TerminalBlock_MetzConnect:TerminalBlock_MetzConnect_Type101_RT01606HBWC_1x06_P5.08mm_Horizontal"
+	(footprint "fp:TerminalBlock_MetzConnect_Type101_RT01606HBWC_1x06_P5.08mm_Horizontal"
 		(layer "F.Cu")
 		(at 132.22 79.67)
@@
 			)
 		)
-		(property "Footprint" "TerminalBlock_MetzConnect:TerminalBlock_MetzConnect_Type101_RT01606HBWC_1x06_P5.08mm_Horizontal"
+		(property "Footprint" "fp:TerminalBlock_MetzConnect_Type101_RT01606HBWC_1x06_P5.08mm_Horizontal"
 			(at 0 0 0)
 			(unlocked yes)
@@
 		)
 	)
-	(footprint "Diode_THT:D_DO-41_SOD81_P10.16mm_Horizontal"
+	(footprint "fp:D_DO-41_SOD81_P10.16mm_Horizontal"
 		(layer "F.Cu")
 		(at 152.19 101.35)
@@
 			)
 		)
-		(property "Footprint" "Diode_THT:D_DO-41_SOD81_P10.16mm_Horizontal"
+		(property "Footprint" "fp:D_DO-41_SOD81_P10.16mm_Horizontal"
 			(at 0 0 0)
 			(unlocked yes)
