File: fsd-amp.kicad_sch (KiCad schematic)
At the start: 13 parts, among them J1001 Screw_Terminal_01x06, J1004 AudioJack2_Ground_Switch, Q1001 FZT 653 ZET, Q1002 FZT 653 ZET, Q1003 FZT 753 ZET

Commit message: export footprints and symbols to project libraries
Parts:
- C1001, C1003: footprint Capacitor_THT:CP_Radial_D10.0mm_P5.00mm -> fp:CP_Radial_D10.0mm_P5.00mm; symbol Device:C_Polarized -> sym:C_Polarized
- C1002: footprint Capacitor_THT:C_Rect_L7.2mm_W11.0mm_P5.00mm_FKS2_FKP2_MKS2_MKP2 -> fp:C_Rect_L7.2mm_W11.0mm_P5.00mm_FKS2_FKP2_MKS2_MKP2; symbol Device:C -> sym:C
- D1001, D1002: footprint Diode_THT:D_DO-41_SOD81_P10.16mm_Horizontal -> fp:D_DO-41_SOD81_P10.16mm_Horizontal; symbol Device:D -> sym:D
- J1001: footprint TerminalBlock_MetzConnect:TerminalBlock_MetzConnect_Type101_RT01606HBWC_1x06_P5.08mm_Horizontal -> fp:TerminalBlock_MetzConnect_Type101_RT01606HBWC_1x06_P5.08mm_Horizontal; symbol Connector:Screw_Terminal_01x06 -> sym:Screw_Terminal_01x06
- J1004: footprint Connector_Audio:Jack_3.5mm_Ledino_KB3SPRS_Horizontal -> fp:Jack_3.5mm_Ledino_KB3SPRS_Horizontal; symbol Connector_Audio:AudioJack2_Ground_Switch -> sym:AudioJack2_Ground_Switch
- Q1001, Q1002: footprint Package_TO_SOT_SMD:SOT-223-3_TabPin2 -> fp:SOT-223-3_TabPin2; symbol Device:Q_NPN_BCE -> sym:Q_NPN_BCE
- Q1003: footprint Package_TO_SOT_SMD:SOT-223-3_TabPin2 -> fp:SOT-223-3_TabPin2; symbol Device:Q_PNP_BCE -> sym:Q_PNP_BCE
- R1001, R1002: footprint Resistor_THT:R_Axial_DIN0207_L6.3mm_D2.5mm_P10.16mm_Horizontal -> fp:R_Axial_DIN0207_L6.3mm_D2.5mm_P10.16mm_Horizontal; symbol Device:R -> sym:R
- RV1001: footprint Potentiometer_THT:Potentiometer_Bourns_3296W_Vertical -> fp:Potentiometer_Bourns_3296W_Vertical; symbol Device:R_Potentiometer -> sym:R_Potentiometer
Changed lines of the file:
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@@
 	)
 	(symbol
-		(lib_id "Connector:Screw_Terminal_01x06")
+		(lib_id "sym:Screw_Terminal_01x06")
 		(at 139.7 171.45 0)
 		(mirror y)
@@
 			)
 		)
-		(property "Footprint" "TerminalBlock_MetzConnect:TerminalBlock_MetzConnect_Type101_RT01606HBWC_1x06_P5.08mm_Horizontal"
+		(property "Footprint" "fp:TerminalBlock_MetzConnect_Type101_RT01606HBWC_1x06_P5.08mm_Horizontal"
 			(at 139.7 171.45 0)
 			(effects
@@
 	)
 	(symbol
-		(lib_id "power:GND")
+		(lib_id "sym:GND")
 		(at 88.9 179.07 0)
 		(unit 1)
@@
 	)
 	(symbol
-		(lib_id "power:PWR_FLAG")
+		(lib_id "sym:PWR_FLAG")
 		(at 146.05 179.07 180)
 		(unit 1)
@@
 	)
 	(symbol
-		(lib_id "Device:Q_PNP_BCE")
+		(lib_id "sym:Q_PNP_BCE")
 		(at 170.18 106.68 0)
 		(mirror x)
@@
 			)
 		)
-		(property "Footprint" "Package_TO_SOT_SMD:SOT-223-3_TabPin2"
+		(property "Footprint" "fp:SOT-223-3_TabPin2"
 			(at 175.26 109.22 0)
 			(effects
@@
 	)
 	(symbol
-		(lib_id "power:+9V")
+		(lib_id "sym:+9V")
 		(at 161.29 176.53 270)
 		(mirror x)
@@
 	)
 	(symbol
-		(lib_id "power:GND")
+		(lib_id "sym:GND")
 		(at 147.32 132.08 0)
 		(unit 1)
@@
 	)
 	(symbol
-		(lib_id "power:GND")
+		(lib_id "sym:GND")
 		(at 147.32 179.07 90)
 		(mirror x)
@@
 	)
 	(symbol
-		(lib_id "Device:R_Potentiometer")
+		(lib_id "sym:R_Potentiometer")
 		(at 114.3 119.38 0)
 		(unit 1)
@@
 			)
 		)
-		(property "Footprint" "Potentiometer_THT:Potentiometer_Bourns_3296W_Vertical"
+		(property "Footprint" "fp:Potentiometer_Bourns_3296W_Vertical"
 			(at 114.3 119.38 0)
 			(effects
@@
 	)
 	(symbol
-		(lib_id "power:GND")
+		(lib_id "sym:GND")
 		(at 121.92 81.28 0)
 		(unit 1)
@@
 	)
 	(symbol
-		(lib_id "Device:Q_NPN_BCE")
+		(lib_id "sym:Q_NPN_BCE")
 		(at 170.18 81.28 0)
 		(unit 1)
@@
 			)
 		)
-		(property "Footprint" "Package_TO_SOT_SMD:SOT-223-3_TabPin2"
+		(property "Footprint" "fp:SOT-223-3_TabPin2"
 			(at 175.26 78.74 0)
 			(effects
@@
 	)
 	(symbol
-		(lib_id "power:GND")
+		(lib_id "sym:GND")
 		(at 144.78 168.91 90)
 		(mirror x)
@@
 	)
 	(symbol
-		(lib_id "Device:R")
+		(lib_id "sym:R")
 		(at 147.32 72.39 0)
 		(unit 1)
@@
 			)
 		)
-		(property "Footprint" "Resistor_THT:R_Axial_DIN0207_L6.3mm_D2.5mm_P10.16mm_Horizontal"
+		(property "Footprint" "fp:R_Axial_DIN0207_L6.3mm_D2.5mm_P10.16mm_Horizontal"
 			(at 145.542 72.39 90)
 			(effects
@@
 	)
 	(symbol
-		(lib_id "Device:C_Polarized")
+		(lib_id "sym:C_Polarized")
 		(at 189.23 93.98 90)
 		(unit 1)
@@
 			)
 		)
-		(property "Footprint" "Capacitor_THT:CP_Radial_D10.0mm_P5.00mm"
+		(property "Footprint" "fp:CP_Radial_D10.0mm_P5.00mm"
 			(at 193.04 93.0148 0)
 			(effects
@@
 	)
 	(symbol
-		(lib_id "Device:Q_NPN_BCE")
+		(lib_id "sym:Q_NPN_BCE")
 		(at 144.78 119.38 0)
 		(unit 1)
@@
 			)
 		)
-		(property "Footprint" "Package_TO_SOT_SMD:SOT-223-3_TabPin2"
+		(property "Footprint" "fp:SOT-223-3_TabPin2"
 			(at 149.86 116.84 0)
 			(effects
@@
 	)
 	(symbol
-		(lib_id "Device:D")
+		(lib_id "sym:D")
 		(at 147.32 87.63 90)
 		(unit 1)
@@
 			)
 		)
-		(property "Footprint" "Diode_THT:D_DO-41_SOD81_P10.16mm_Horizontal"
+		(property "Footprint" "fp:D_DO-41_SOD81_P10.16mm_Horizontal"
 			(at 147.32 87.63 0)
 			(effects
@@
 	)
 	(symbol
-		(lib_id "power:+9V")
+		(lib_id "sym:+9V")
 		(at 147.32 62.23 0)
 		(unit 1)
@@
 	)
 	(symbol
-		(lib_id "power:GND")
+		(lib_id "sym:GND")
 		(at 144.78 173.99 90)
 		(mirror x)
@@
 	)
 	(symbol
-		(lib_id "Connector_Audio:AudioJack2_Ground_Switch")
+		(lib_id "sym:AudioJack2_Ground_Switch")
 		(at 88.9 171.45 0)
 		(unit 1)
@@
 			)
 		)
-		(property "Footprint" "Connector_Audio:Jack_3.5mm_Ledino_KB3SPRS_Horizontal"
+		(property "Footprint" "fp:Jack_3.5mm_Ledino_KB3SPRS_Horizontal"
 			(at 88.9 166.37 0)
 			(effects
@@
 	)
 	(symbol
-		(lib_id "Device:R")
+		(lib_id "sym:R")
 		(at 134.62 113.03 0)
 		(unit 1)
@@
 			)
 		)
-		(property "Footprint" "Resistor_THT:R_Axial_DIN0207_L6.3mm_D2.5mm_P10.16mm_Horizontal"
+		(property "Footprint" "fp:R_Axial_DIN0207_L6.3mm_D2.5mm_P10.16mm_Horizontal"
 			(at 132.842 113.03 90)
 			(effects
@@
 	)
 	(symbol
-		(lib_id "Device:C")
+		(lib_id "sym:C")
 		(at 125.73 119.38 90)
 		(unit 1)
@@
 			)
 		)
-		(property "Footprint" "Capacitor_THT:C_Rect_L7.2mm_W11.0mm_P5.00mm_FKS2_FKP2_MKS2_MKP2"
+		(property "Footprint" "fp:C_Rect_L7.2mm_W11.0mm_P5.00mm_FKS2_FKP2_MKS2_MKP2"
 			(at 129.54 118.4148 0)
 			(effects
@@
 	)
 	(symbol
-		(lib_id "Device:D")
+		(lib_id "sym:D")
 		(at 147.32 100.33 90)
 		(unit 1)
@@
 			)
 		)
-		(property "Footprint" "Diode_THT:D_DO-41_SOD81_P10.16mm_Horizontal"
+		(property "Footprint" "fp:D_DO-41_SOD81_P10.16mm_Horizontal"
 			(at 147.32 100.33 0)
 			(effects
@@
 	)
 	(symbol
-		(lib_id "Device:C_Polarized")
+		(lib_id "sym:C_Polarized")
 		(at 121.92 72.39 0)
 		(unit 1)
@@
 			)
 		)
-		(property "Footprint" "Capacitor_THT:CP_Radial_D10.0mm_P5.00mm"
+		(property "Footprint" "fp:CP_Radial_D10.0mm_P5.00mm"
 			(at 122.8852 76.2 0)
 			(effects
@@
 	)
 	(symbol
-		(lib_id "power:PWR_FLAG")
+		(lib_id "sym:PWR_FLAG")
 		(at 160.02 176.53 180)
 		(unit 1)
